Commit message: gazebo model shows. but not moving yet

File: src/manipulator/urdf/model.urdf.xacro (robot description, xacro)
@@ -2,4 +2,13 @@
 <robot xmlns:xacro="http://www.ros.org/wiki/xacro" name="5dof_robot_manipulator">
     <xacro:include filename="inertial_macros.xacro"/>
+    <!-- <xacro:include filename="gazebo_control.xacro"/> -->
+    <!-- <gazebo>
+        <plugin name="gazebo_ros2_control" filename="libgazebo_ros2_control.so"/>
+    </gazebo> -->
+    <gazebo>
+        <plugin name="gazebo_ros2_control" filename="libgazebo_ros2_control.so">
+            <parameters>/home/bgb_6342/ws_manipulator/src/manipulator/config/ros2_controllers.yaml</parameters>
+        </plugin>
+    </gazebo>
     <!-- COLOR DEFINITIONS -->
     <material name="blue">
@@ -25,5 +34,5 @@
     <link name="world"/>
     <joint name="fixed_joint" type="fixed">
-        <origin rpy="0 0 0" xyz="0 0 0" />
+        <origin rpy="0 0 0" xyz="0 0 0.1" />
         <parent link="world"/>
         <child link="base_link"/>
@@ -47,4 +56,7 @@
         </xacro:inertial_cylinder>
     </link>
+    <gazebo reference="base_link">
+        <material>Gazebo/Black</material>
+    </gazebo>
     <joint name="joint_1" type="revolute">
         <parent link="base_link"/>
@@ -72,4 +84,7 @@
         </xacro:inertial_cylinder>
     </link>
+    <gazebo reference="link_1">
+        <material>Gazebo/Blue</material>
+    </gazebo>
     <joint name="joint_2" type="revolute">
         <parent link="link_1"/>
@@ -97,4 +112,7 @@
         </xacro:inertial_cylinder>
     </link>
+    <gazebo reference="link_2">
+        <material>Gazebo/Grey</material>
+    </gazebo>
     <joint name="joint_3" type="revolute">
         <parent link="link_2"/>
@@ -122,4 +140,7 @@
         </xacro:inertial_cylinder>
     </link>
+    <gazebo reference="link_3">
+        <material>Gazebo/Blue</material>
+    </gazebo>
     <joint name="joint_4" type="revolute">
         <parent link="link_3"/>
@@ -147,4 +168,7 @@
         </xacro:inertial_cylinder>
     </link>
+    <gazebo reference="link_4">
+        <material>Gazebo/Grey</material>
+    </gazebo>
     <joint name="joint_5" type="revolute">
         <parent link="link_4"/>
@@ -172,3 +196,36 @@
         </xacro:inertial_cylinder>
     </link>
+    <gazebo reference="link_5">
+        <material>Gazebo/Blue</material>
+    </gazebo>
+    <ros2_control name="GazeboSystem" type="system">
+        <hardware>
+            <plugin>gazebo_ros2_control/GazeboSystem</plugin>
+        </hardware>
+        <joint name="joint_1">
+                <command_interface name="position"/>
+                <state_interface name="position"/>
+                <state_interface name="velocity"/>
+        </joint>
+        <joint name="joint_2">
+            <command_interface name="position"/>
+            <state_interface name="position"/>
+            <state_interface name="velocity"/>
+        </joint>
+        <joint name="joint_3">
+            <command_interface name="position"/>
+            <state_interface name="position"/>
+            <state_interface name="velocity"/>
+        </joint>
+        <joint name="joint_4">
+            <command_interface name="position"/>
+            <state_interface name="position"/>
+            <state_interface name="velocity"/>
+        </joint>
+        <joint name="joint_5">
+            <command_interface name="position"/>
+            <state_interface name="position"/>
+            <state_interface name="velocity"/>
+        </joint>
+    </ros2_control>
 </robot>
